File: pcb/MarsRover.kicad_sch (KiCad schematic)
At the start: 38 parts, among them J2 JST-PH 2,0, M1 Vibrationsmotor L, M2 Vibrationsmotor R, Q1 AO3400A, Q2 AO3400A, U1 ESP32-DevKitC V4, U2 TP4056-Modul, U5 MT3608 auf 5,00V, U6 GY-521 MPU-6050, U7 GY-530 VL53L0X

Commit message: Schaltplan neu aufgebaut: fuenf Bereiche, 175 gezeichnete Leitungen
Der alte Schaltplan verband alles ueber Netzlabels, die Bauteile standen
ungeordnet auf dem Blatt. Jetzt:

  Blatt A2, fuenf beschriftete Bereiche -- Rechenkern, Motortreiber,
  Sensoren Linienerkennung, Sensoren Lage und Abstand, Signal-LEDs,
  Akku und Ladevorrichtung.
  175 gezeichnete Leitungen, 25 Knotenpunkte, NULL Netzlabels.

Geprueft: ERC 0 Fehler, keine verwaisten Leitungen, keine Ueberlappungen,
Netzliste knotengenau gegen den Entwurf abgeglichen. Zwei echte
Zeichenfehler behoben -- Leitungen liefen durch die Gehaeuse von U2 und U5.

Die LED-MOSFETs entfallen wieder: ESP32-WROOM-32 v3.8, Tabelle 14 nennt
I_OH typisch 40 mA je Pin in der Domaene VDD3P3_RTC, bei mehreren
treibenden Pins noch rund 29 mA. Alle vier LED-Pins liegen dort.
Vorwiderstand bleibt 220 Ohm. Spart zwoelf Bauteile.

build_schematic.py loest gen_schematic.py ab; die acht Lagen sind am
lebenden KiCad ausgemessen, und das Skript prueft selbst, ob jede
Koordinate auf dem 1,27-mm-Raster liegt. gen_schematic.py ist gesperrt,
damit ein versehentlicher Lauf den Schaltplan nicht ueberschreibt.

Co-Authored-By: Claude Opus 5 <noreply@anthropic.com>
Parts:
- LED1: value gelb -> gelb - vorne links
- LED2: value gelb -> gelb - vorne rechts
- LED3: value rot -> rot - hinten links
- LED4: value rot -> rot - hinten rechts
- M1: value Vibrationsmotor L -> Vibrationsmotor links
- M2: value Vibrationsmotor R -> Vibrationsmotor rechts
- OS1: value TCRT5000 -> TCRT5000 links
- OS2: value TCRT5000 -> TCRT5000 rechts
Connections:
- net +5V: now also D1.1 (K), D2.1 (K); no longer D1.2 (A), D2.2 (A)
- net I2C_SCL: no longer names the net of U1.36 (GPIO22), U6.3 (Pin_3), U7.3 (Pin_3)
- net I2C_SDA: no longer names the net of U1.33 (GPIO21), U6.4 (Pin_4), U7.4 (Pin_4)
- net LED_FL: no longer names the net of R9.1, U1.12 (MTMS/GPIO14/ADC2_CH6)
- net LED_FL_A: no longer names the net of LED1.2 (A), R9.2
- net LED_FR: no longer names the net of R10.1, U1.11 (ADC2_CH7/GPIO27)
- net LED_FR_A: no longer names the net of LED2.2 (A), R10.2
- net LED_RL: no longer names the net of R11.1, U1.10 (DAC_2/ADC2_CH9/GPIO26)
- net LED_RL_A: no longer names the net of LED3.2 (A), R11.2
- net LED_RR: no longer names the net of R12.1, U1.9 (DAC_1/ADC2_CH8/GPIO25)
- net LED_RR_A: no longer names the net of LED4.2 (A), R12.2
- net LINE_L: no longer names the net of OS1.4 (E), R7.1, U1.5 (VDET_1/GPIO34/ADC1_CH6)
- net LINE_R: no longer names the net of OS2.4 (E), R8.1, U1.6 (VDET_2/GPIO35/ADC1_CH7)
- net LS_L_A: no longer names the net of OS1.1 (A), R5.2
- net LS_R_A: no longer names the net of OS2.1 (A), R6.2
- net MOT_L_D: no longer names the net of C3.1, M1.2 (-), Q1.3 (D)
- net MOT_L_D: now also D1.2 (A); no longer D1.1 (K)
- net MOT_L_G: no longer names the net of R1.1, U1.7 (32K_XP/GPIO32/ADC1_CH4)
- net MOT_L_GT: no longer names the net of Q1.1 (G), R1.2, R3.1
- net MOT_R_D: no longer names the net of C4.1, M2.2 (-), Q2.3 (D)
- net MOT_R_D: now also D2.2 (A); no longer D2.1 (K)
- net MOT_R_G: no longer names the net of R2.1, U1.8 (32K_XN/GPIO33/ADC1_CH5)
- net MOT_R_GT: no longer names the net of Q2.1 (G), R2.2, R4.1
- net USB_VBUS: no longer names the net of U2.1 (Pin_1)
- net VBAT_PROT: no longer names the net of R16.1, S1.2 (B), U2.5 (Pin_5)
- net VBAT_RAW: no longer names the net of BT1.1 (+), J2.1 (Pin_1), U2.3 (Pin_3)
- net VBAT_SENSE: no longer names the net of R16.2, R17.1, U1.4 (SENSOR_VN/GPIO39/ADC1_CH3)
- net VBAT_SW: no longer names the net of S1.1 (A), U5.1 (Pin_1)
- no-connect marks 23 -> 24
Other:
- note added: "AKKU UND LADEVORRICHTUNG"
- note added: "MOTORTREIBER"
- note added: "RECHENKERN"
- note added: "SENSOREN Lage und Abstand"
- note added: "SENSOREN Linienerkennung"
- note added: "SIGNAL-LEDS"
- note added: "USB-C-Buchse sitzt auf dem TP4056-Fertigmodul,"
- note added: "nicht auf dieser Platine"
