File: pcb/MarsRover.kicad_sch (KiCad schematic)
At the start: 38 parts, among them J2 JST-PH 2,0, M1 Vibrationsmotor links, M2 Vibrationsmotor rechts, Q1 AO3400A, Q2 AO3400A, U1 ESP32-DevKitC V4, U2 TP4056-Modul, U5 MT3608 auf 5,00V, U6 GY-521 MPU-6050, U7 GY-530 VL53L0X

Commit message: Entkopplung ergaenzt: C5 bis C12, Motoranschluesse als Loetaugen
Neu, alle mit gezeichneten Leitungen eingefuegt:

  C5   100n     parallel zu C1/C2 an der 5-V-Schiene
  C6   10u/25V  am ESP32, VIN gegen Masse
  C7   100n     am ESP32, VIN gegen Masse
  C8   100n     am ESP32, 3V3 gegen Masse
  C9   100n     an OS1
  C10  100n     an OS2
  C11  47u/10V  an der linken Motorstufe, +5V gegen Masse
  C12  47u/10V  an der rechten Motorstufe, +5V gegen Masse

Geaendert:
  C1   100u/16V -> 100u/10V   Alu-Elko, zweifache Reserve reicht
  C2   10u      -> 10u/25V    Keramik: 10 V waere falsch herum gedacht,
                              ein X5R/X7R verliert unter Gleichspannung
                              Kapazitaet. Mit 25 V statt 10 V bleibt im
                              selben Gehaeuse deutlich mehr uebrig.

Die 47 uF liegen NICHT ueber den Motorklemmen, sondern von +5V nach
Masse an der jeweiligen Stufe. Ueber den Klemmen wuerde der Elko bei
jedem PWM-Takt ueber den MOSFET entladen -- 20 000 Stoesse je Sekunde,
weit jenseits des Rippelstroms, den ein 47-uF-Elko vertraegt, und eine
unnoetige Belastung des AO3400A. Von +5V nach Masse erfuellt er denselben
Zweck: er liefert den Stromimpuls oertlich und haelt ihn aus dem Rest
der Platine heraus, wo das ADC-Frontend sitzt.

Weggelassen gegenueber dem Vorschlag: 1 uF an den Sensoren (die TCRT5000
schalten nichts, 8 mA Gleichstrom) und 10 uF an 3,3 V (den Bulk bringt
der AMS1117 des DevKits schon mit).

M1 und M2 bekommen den Fussabdruck PinHeader_1x02_P2.54mm_Vertical --
zwei durchkontaktierte Loecher mit 1,0 mm als Loetaugen, weil die Motoren
abgesetzt sitzen. Dazu ein Hinweis auf dem Blatt.

Geprueft: ERC 0 Fehler, keine Ueberlappungen, Netzliste 51 Netze wie
zuvor, alle zwoelf Kondensatoren an den richtigen Netzen.

Co-Authored-By: Claude Opus 5 <noreply@anthropic.com>
Parts:
- added C10, C5, C7, C8, C9: 100n, symbol Device:C
- added C11, C12: 47u/10V, symbol Device:C_Polarized
- added C6: 10u/25V, symbol Device:C
- C1: value 100u/16V -> 100u/10V
- C2: value 10u -> 10u/25V
- M1, M2: footprint (none) -> Connector_PinHeader_2.54mm:PinHeader_1x02_P2.54mm_Vertical; Hinweis (none) -> Motor sitzt abgesetzt, Anschluss ueber zwei Loetaugen
Connections:
- net +3V3: now also C10.1, C8.1, C9.1
- net +5V: now also C11.1, C12.1, C5.1, C6.1, C7.1
- net GND: now also C10.2, C11.2, C12.2, C5.2, C6.2, C7.2, C8.2, C9.2
Other:
- note added: "Fussabdruck PinHeader_1x02_P2.54mm_Vertical, Litze direkt einloeten."
- note added: "Motoren sitzen abgesetzt. Auf der Platine je zwei Loetaugen,"

Commit message: Stueckliste nachgezogen, Fussabdruecke fuer alle Bauteile zugewiesen
Stueckliste:
  - Rechenkern war noch auf DevKit V1 30-Pin, jetzt DevKitC V4 38-Pin
  - C1 auf 100u/10V, C2 auf 10u/25V, C5 neu
  - neuer Abschnitt 5a Entkopplung mit C6 bis C10
  - C11/C12 im Motortreiber, samt Begruendung warum sie nach GND gehen
    und nicht ueber die Motorklemmen
  - Loetaugen fuer M1/M2 als eigene Position
  - LED-Abschnitt: Datenblattbeleg, warum kein MOSFET noetig ist
  - Kosten neu: 27,10 EUR, mit I2C-Sensorik 34,20 EUR

Fussabdruecke, Aufteilung nach Stueckliste -- 0805 fuer Gate- und
Entkopplungskram, bedrahtet fuer alles von Hand zu Justierende:

  U1          PCM_Espressif:ESP32-DevKitC (38 Pads, Umriss 27,9 x 47,4 mm)
  U2/U5/U6/U7 Stiftleisten 1x06 bzw. 1x04 (Fertigmodule)
  M1/M2       PinHeader_1x02 als Loetaugen, Motoren sitzen abgesetzt
  OS1/OS2     OptoDevice:Vishay_TCRT5000
  Q1/Q2       SOT-23,  D1/D2 DO-41,  LED1-4 3 mm
  R1-R4       0805,    R5-R12/R16/R17 bedrahtet
  C2-C10      0805,    C1 Elko 6,3 mm, C11/C12 Elko 5 mm
  BT1         ohne Fussabdruck, als "nicht auf der Platine" markiert

Geprueft: 45 von 46 Bauteilen mit Fussabdruck, Netzliste unveraendert
bei 51 Netzen.

Co-Authored-By: Claude Opus 5 <noreply@anthropic.com>
Parts:
- C1: footprint (none) -> Capacitor_THT:CP_Radial_D6.3mm_P2.50mm
- C10, C2, C3, C4, C5, C6, C7, C8, C9: footprint (none) -> Capacitor_SMD:C_0805_2012Metric
- C11, C12: footprint (none) -> Capacitor_THT:CP_Radial_D5.0mm_P2.00mm
- D1, D2: footprint (none) -> Diode_THT:D_DO-41_SOD81_P7.62mm_Horizontal
- J2: footprint (none) -> Connector_JST:JST_PH_B2B-PH-K_1x02_P2.00mm_Vertical
- LED1, LED2, LED3, LED4: footprint (none) -> LED_THT:LED_D3.0mm
- OS1, OS2: footprint (none) -> OptoDevice:Vishay_TCRT5000
- Q1, Q2: footprint (none) -> Package_TO_SOT_SMD:SOT-23
- R1, R2, R3, R4: footprint (none) -> Resistor_SMD:R_0805_2012Metric
- R10, R11, R12, R16, R17, R5, R6, R7, R8, R9: footprint (none) -> Resistor_THT:R_Axial_DIN0207_L6.3mm_D2.5mm_P7.62mm_Horizontal
- S1: footprint (none) -> Button_Switch_THT:SW_Slide_SPDT_Straight_CK_OS102011MS2Q
- U1: footprint (none) -> PCM_Espressif:ESP32-DevKitC
- U2: footprint (none) -> Connector_PinHeader_2.54mm:PinHeader_1x06_P2.54mm_Vertical
- U5, U6, U7: footprint (none) -> Connector_PinHeader_2.54mm:PinHeader_1x04_P2.54mm_Vertical
Changed lines of the file:
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@@
 			)
 		)
-		(property "Footprint" ""
+		(property "Footprint" "Diode_THT:D_DO-41_SOD81_P7.62mm_Horizontal"
 			(at 142.24 46.99 0)
 			(hide yes)
@@
 			)
 		)
-		(property "Footprint" ""
+		(property "Footprint" "Button_Switch_THT:SW_Slide_SPDT_Straight_CK_OS102011MS2Q"
 			(at 132.08 309.88 0)
 			(hide yes)
@@
 			)
 		)
-		(property "Footprint" ""
+		(property "Footprint" "Capacitor_SMD:C_0805_2012Metric"
 			(at 177.8 134.62 0)
 			(hide yes)
@@
 			)
 		)
-		(property "Footprint" ""
+		(property "Footprint" "Package_TO_SOT_SMD:SOT-23"
 			(at 157.48 139.7 0)
 			(hide yes)
@@
 			)
 		)
-		(property "Footprint" ""
+		(property "Footprint" "Resistor_THT:R_Axial_DIN0207_L6.3mm_D2.5mm_P7.62mm_Horizontal"
 			(at 76.2 322.58 0)
 			(hide yes)
@@
 			)
 		)
-		(property "Footprint" ""
+		(property "Footprint" "Resistor_THT:R_Axial_DIN0207_L6.3mm_D2.5mm_P7.62mm_Horizontal"
 			(at 414.02 203.2 0)
 			(hide yes)
@@
 			)
 		)
-		(property "Footprint" ""
+		(property "Footprint" "LED_THT:LED_D3.0mm"
 			(at 433.07 215.9 0)
 			(hide yes)
@@
 			)
 		)
-		(property "Footprint" ""
+		(property "Footprint" "OptoDevice:Vishay_TCRT5000"
 			(at 152.4 215.9 0)
 			(hide yes)
@@
 			)
 		)
-		(property "Footprint" ""
+		(property "Footprint" "Connector_PinHeader_2.54mm:PinHeader_1x04_P2.54mm_Vertical"
 			(at 360.68 127 0)
 			(hide yes)
@@
 			)
 		)
-		(property "Footprint" ""
+		(property "Footprint" "Diode_THT:D_DO-41_SOD81_P7.62mm_Horizontal"
 			(at 142.24 115.57 0)
 			(hide yes)
@@
 			)
 		)
-		(property "Footprint" ""
+		(property "Footprint" "Resistor_THT:R_Axial_DIN0207_L6.3mm_D2.5mm_P7.62mm_Horizontal"
 			(at 114.3 240.03 0)
 			(hide yes)
@@
 			)
 		)
-		(property "Footprint" ""
+		(property "Footprint" "Resistor_SMD:R_0805_2012Metric"
 			(at 133.35 139.7 0)
 			(hide yes)
@@
 			)
 		)
-		(property "Footprint" ""
+		(property "Footprint" "Resistor_THT:R_Axial_DIN0207_L6.3mm_D2.5mm_P7.62mm_Horizontal"
 			(at 414.02 177.8 0)
 			(hide yes)
@@
 			)
 		)
-		(property "Footprint" ""
+		(property "Footprint" "Capacitor_SMD:C_0805_2012Metric"
 			(at 177.8 66.04 0)
 			(hide yes)
@@
 			)
 		)
-		(property "Footprint" ""
+		(property "Footprint" "PCM_Espressif:ESP32-DevKitC"
 			(at 274.32 109.22 0)
 			(hide yes)
@@
 		(exclude_from_sim no)
 		(in_bom yes)
-		(on_board yes)
+		(on_board no)
 		(in_pos_files yes)
 		(dnp no)
@@
 			)
 		)
-		(property "Footprint" ""
+		(property "Footprint" "LED_THT:LED_D3.0mm"
 			(at 433.07 190.5 0)
 			(hide yes)
@@
 			)
 		)
-		(property "Footprint" ""
+		(property "Footprint" "Resistor_THT:R_Axial_DIN0207_L6.3mm_D2.5mm_P7.62mm_Horizontal"
 			(at 109.22 196.85 0)
 			(hide yes)
@@
 			)
 		)
-		(property "Footprint" ""
+		(property "Footprint" "Resistor_SMD:R_0805_2012Metric"
 			(at 144.78 147.32 0)
 			(hide yes)
@@
 			)
 		)
-		(property "Footprint" ""
+		(property "Footprint" "Resistor_THT:R_Axial_DIN0207_L6.3mm_D2.5mm_P7.62mm_Horizontal"
 			(at 414.02 190.5 0)
 			(hide yes)
@@
 			)
 		)
-		(property "Footprint" ""
+		(property "Footprint" "Resistor_THT:R_Axial_DIN0207_L6.3mm_D2.5mm_P7.62mm_Horizontal"
 			(at 414.02 215.9 0)
 			(hide yes)
@@
 			)
 		)
-		(property "Footprint" ""
+		(property "Footprint" "Connector_PinHeader_2.54mm:PinHeader_1x06_P2.54mm_Vertical"
 			(at 104.14 304.8 0)
 			(hide yes)
@@
 			)
 		)
-		(property "Footprint" ""
+		(property "Footprint" "LED_THT:LED_D3.0mm"
 			(at 433.07 177.8 0)
 			(hide yes)
@@
 			)
 		)
-		(property "Footprint" ""
+		(property "Footprint" "Resistor_SMD:R_0805_2012Metric"
 			(at 133.35 71.12 0)
 			(hide yes)
@@
 			)
 		)
-		(property "Footprint" ""
+		(property "Footprint" "OptoDevice:Vishay_TCRT5000"
 			(at 111.76 214.63 0)
 			(hide yes)
@@
 			)
 		)
-		(property "Footprint" ""
+		(property "Footprint" "Resistor_THT:R_Axial_DIN0207_L6.3mm_D2.5mm_P7.62mm_Horizontal"
 			(at 76.2 340.36 0)
 			(hide yes)
@@
 			)
 		)
-		(property "Footprint" ""
+		(property "Footprint" "Package_TO_SOT_SMD:SOT-23"
 			(at 157.48 71.12 0)
 			(hide yes)
@@
 			)
 		)
-		(property "Footprint" ""
+		(property "Footprint" "Capacitor_THT:CP_Radial_D6.3mm_P2.50mm"
 			(at 182.88 326.39 0)
 			(hide yes)
@@
 			)
 		)
-		(property "Footprint" ""
+		(property "Footprint" "Resistor_THT:R_Axial_DIN0207_L6.3mm_D2.5mm_P7.62mm_Horizontal"
 			(at 154.94 241.3 0)
 			(hide yes)
@@
 			)
 		)
-		(property "Footprint" ""
+		(property "Footprint" "Resistor_SMD:R_0805_2012Metric"
 			(at 144.78 78.74 0)
 			(hide yes)
@@
 			)
 		)
-		(property "Footprint" ""
+		(property "Footprint" "Connector_JST:JST_PH_B2B-PH-K_1x02_P2.00mm_Vertical"
 			(at 66.04 287.02 0)
 			(hide yes)
@@
 			)
 		)
-		(property "Footprint" ""
+		(property "Footprint" "Resistor_THT:R_Axial_DIN0207_L6.3mm_D2.5mm_P7.62mm_Horizontal"
 			(at 149.86 198.12 0)
 			(hide yes)
@@
 			)
 		)
-		(property "Footprint" ""
+		(property "Footprint" "Connector_PinHeader_2.54mm:PinHeader_1x04_P2.54mm_Vertical"
 			(at 360.68 91.44 0)
 			(hide yes)
@@
 			)
 		)
-		(property "Footprint" ""
+		(property "Footprint" "Connector_PinHeader_2.54mm:PinHeader_1x04_P2.54mm_Vertical"
 			(at 167.64 307.34 0)
 			(hide yes)
@@
 			)
 		)
-		(property "Footprint" ""
+		(property "Footprint" "Capacitor_SMD:C_0805_2012Metric"
 			(at 203.2 326.39 0)
 			(hide yes)
@@
 			)
 		)
-		(property "Footprint" ""
+		(property "Footprint" "LED_THT:LED_D3.0mm"
 			(at 433.07 203.2 0)
 			(hide yes)
@@
 			)
 		)
-		(property "Footprint" ""
+		(property "Footprint" "Capacitor_SMD:C_0805_2012Metric"
 			(at 213.36 326.39 0)
 			(hide yes)
@@
 			)
 		)
-		(property "Footprint" ""
+		(property "Footprint" "Capacitor_SMD:C_0805_2012Metric"
 			(at 250.19 45.72 0)
 			(hide yes)
@@
 			)
 		)
-		(property "Footprint" ""
+		(property "Footprint" "Capacitor_SMD:C_0805_2012Metric"
 			(at 266.70 45.72 0)
 			(hide yes)
@@
 			)
 		)
-		(property "Footprint" ""
+		(property "Footprint" "Capacitor_SMD:C_0805_2012Metric"
 			(at 283.21 45.72 0)
 			(hide yes)
@@
 			)
 		)
-		(property "Footprint" ""
+		(property "Footprint" "Capacitor_SMD:C_0805_2012Metric"
 			(at 99.06 214.63 0)
 			(hide yes)
@@
 			)
 		)
-		(property "Footprint" ""
+		(property "Footprint" "Capacitor_SMD:C_0805_2012Metric"
 			(at 139.70 215.90 0)
 			(hide yes)
@@
 			)
 		)
-		(property "Footprint" ""
+		(property "Footprint" "Capacitor_THT:CP_Radial_D5.0mm_P2.00mm"
 			(at 189.23 46.99 0)
 			(hide yes)
@@
 			)
 		)
-		(property "Footprint" ""
+		(property "Footprint" "Capacitor_THT:CP_Radial_D5.0mm_P2.00mm"
 			(at 189.23 115.57 0)
 			(hide yes)

Commit message: Platine geroutet: 27 von 27 Netzen, null unverbundene Elemente
Geroutet mit KiCadRoutingTools (A*-Router mit Rust-Kern, MIT, headless auf
der .kicad_pcb). 101 Durchkontaktierungen, Massflaeche auf B.Cu als eine
zusammenhaengende Insel. DRC: 0 Abstandsverstoesse, 0 Kurzschluesse,
0 unverbundene Elemente; es bleiben nur Siebdruck-Kosmetik und die
gewollten Courtyard-Ueberlappungen unter dem gesockelten DevKit.

Platzierung nachgezogen:
- J2 liegend (S2B-PH-K) auf die Unterseite, der Akku kommt darunter
- OS1/OS2 Fototransistoren nach innen, optische Messflecken 18 mm
  auseinander -- im Fenster 15..20 mm fuer ein 19-mm-Band
- U6 hinten mittig, waagerecht montierbar, Gyro-Z bleibt die Hochachse
- S1 daneben
- R2 und Q2 nach aussen: R2 Pad 1 hatte beidseitig nur 0,8 mm Padabstand,
  genau die Breite einer 0,4-mm-Leitung mit Abstand -- daran scheiterten
  zwei Router nacheinander

Kein Ausschnitt fuer den MPU-6050: ein Gyro misst die Drehrate ueberall
gleich, und die Zentrifugalterme liegen bei 0,03 g, zwei Groessenordnungen
unter der Motorvibration. Das Loch haette Steifigkeit und Massflaeche
gekostet, ohne messbar etwas zu bringen.

Netzklassen gesetzt: Default 0,4 mm / Leistung 1,0 mm, Abstand 0,2 mm.

Co-Authored-By: Claude Opus 5 <noreply@anthropic.com>
Parts:
- J2: footprint Connector_JST:JST_PH_B2B-PH-K_1x02_P2.00mm_Vertical -> Connector_JST:JST_PH_S2B-PH-K_1x02_P2.00mm_Horizontal
- R1, R2, R3, R4: footprint Resistor_SMD:R_0805_2012Metric -> Resistor_SMD:R_0805_2012Metric_Pad1.20x1.40mm_HandSolder
- R16, R17, R5, R6, R7, R8: footprint Resistor_THT:R_Axial_DIN0207_L6.3mm_D2.5mm_P7.62mm_Horizontal -> Resistor_SMD:R_0805_2012Metric_Pad1.20x1.40mm_HandSolder
